Commit message: 修复base.urdf.xacro中car的file模式

File: src/four_wheeled_vehicle/urdf/vehicle/base.urdf.xacro (robot description, xacro)
@@ -16,5 +16,5 @@
                 <origin xyz="0 0 0" rpy="0 0 0"/>
                 <geometry>
-                    <mesh filename="file:///home/wu/code/ros2/Pure-tracking-slam-automatic-navigation-system/src/four_wheeled_vehicle/models/four_wheeled_vehicle/meshes/car.dae"/>
+                    <mesh filename="file:///home/wu/code/ros2/Pure-tracking-slam-automatic-navigation-system/src/four_wheeled_vehicle/models/four_wheeled_vehicle/meshes/car.dae" scale="1 1 1"/>
                 </geometry>
             </visual>

Commit message: 添加base_footprint这个link,并且作为base_link的子,这样可以在最大程度上不修改代码,并且能够在rviz中将车放在地面

File: src/four_wheeled_vehicle/urdf/vehicle/base.urdf.xacro (robot description, xacro)
@@ -20,19 +20,9 @@
             </visual>
         </link>
-        <link name="inertial_joint">
-            <origin xyz="0 0 0" rpy="0 0 0"/>
-        </link>
-        <joint name="inertial_joint_fixed" type="fixed">
+        <link name="base_footprint"/>
+        <joint name="base_footprint_joint" type="fixed">
             <parent link="base_link"/>
-            <child link="inertial_joint"/>
-            <origin xyz="0 0 0" rpy="0 0 0"/>
-        </joint>
-        <link name="main_mass">
-            <origin xyz="0 0 0" rpy="0 0 0"/>
-        </link>
-        <joint name="main_mass_fixed" type="fixed">
-            <parent link="inertial_joint"/>
-            <child link="main_mass"/>
-            <origin xyz="0 0 0" rpy="0 0 0"/>
+            <child link="base_footprint"/>
+            <origin xyz="0 0 -0.325" rpy="0 0 0"/>
         </joint>
     </xacro:macro>

Commit message: 修复两个问题见修改.md的1-2

File: src/four_wheeled_vehicle/urdf/vehicle/base.urdf.xacro (robot description, xacro)
@@ -20,10 +20,10 @@
             </visual>
         </link>
-        <link name="base_footprint"/>
+        <!-- <link name="base_footprint"/>
         <joint name="base_footprint_joint" type="fixed">
             <parent link="base_link"/>
             <child link="base_footprint"/>
             <origin xyz="0 0 -0.325" rpy="0 0 0"/>
-        </joint>
+        </joint> -->
     </xacro:macro>
 </robot>

File: src/four_wheeled_vehicle/urdf/vehicle/sensor/laser.urdf.xacro (robot description, xacro)
@@ -11,5 +11,5 @@
             <sensor type="ray" name="laser">
                 <always_on>true</always_on>
-                <update_rate>10</update_rate>
+                <update_rate>5</update_rate>
                 <visualize>true</visualize>
                 <ray>

Commit message: 按照默认的slam_toolbox标准,base设为base_footprint

File: src/four_wheeled_vehicle/urdf/vehicle/base.urdf.xacro (robot description, xacro)
@@ -20,10 +20,10 @@
             </visual>
         </link>
-        <!-- <link name="base_footprint"/>
+        <link name="base_footprint"/>
         <joint name="base_footprint_joint" type="fixed">
-            <parent link="base_link"/>
-            <child link="base_footprint"/>
-            <origin xyz="0 0 -0.325" rpy="0 0 0"/>
-        </joint> -->
+            <parent link="base_footprint"/>
+            <child link="base_link"/>
+            <origin xyz="0 0 0.325" rpy="0 0 0"/>
+        </joint>
     </xacro:macro>
 </robot>

File: src/four_wheeled_vehicle/urdf/vehicle/sensor/lidar3d.urdf.xacro (robot description, xacro)
@@ -44,4 +44,5 @@
                         <remapping>~/out:=/points_raw</remapping>
                     </ros>
+                    <output_type>sensor_msgs/PointCloud2</output_type>
                     <frame_name>lidar3d_link</frame_name>
                 </plugin>

Commit message: 采用阿克曼模型对应的nav2_params,但是参数还是需要调整

File: src/four_wheeled_vehicle/urdf/vehicle/base.urdf.xacro (robot description, xacro)
@@ -10,5 +10,5 @@
                 <origin xyz="0 0 0" rpy="0 0 0"/>
                 <geometry>
-                    <box size="5.24 1.5 0.47"/>
+                    <box size="5.07 1.97 0.47"/>
                 </geometry>
             </collision>
