Commit message: 代码将dae的图片路径进行修改(把xxx.xxx.xxx.jpg改为了xxx_xxx_xxx.jpg)，dae通过file的模式硬编码识别，才能解决rviz加载不了模型的问题。

File: src/four_wheeled_vehicle/urdf/vehicle/actuator/wheel.urdf.xacro (robot description, xacro)
@@ -29,5 +29,5 @@
                 <origin xyz="0 0 0" rpy="0 0 0"/>
                 <geometry>
-                    <mesh filename="model://four_wheeled_vehicle/meshes/wheel_l.dae" scale="1 1 1"/>
+                    <mesh filename="file:///home/wu/code/ros2/Pure-tracking-slam-automatic-navigation-system/src/four_wheeled_vehicle/models/four_wheeled_vehicle/meshes/wheel_l.dae"/>
                 </geometry>
             </visual>
@@ -63,5 +63,5 @@
                 <origin xyz="0 0 0" rpy="0 0 0"/>
                 <geometry>
-                    <mesh filename="model://four_wheeled_vehicle/meshes/wheel_r.dae" scale="1 1 1"/>
+                    <mesh filename="file:///home/wu/code/ros2/Pure-tracking-slam-automatic-navigation-system/src/four_wheeled_vehicle/models/four_wheeled_vehicle/meshes/wheel_r.dae"/>
                 </geometry>
             </visual>

File: src/four_wheeled_vehicle/urdf/vehicle/base.urdf.xacro (robot description, xacro)
@@ -16,5 +16,5 @@
                 <origin xyz="0 0 0" rpy="0 0 0"/>
                 <geometry>
-                    <mesh filename="model://four_wheeled_vehicle/meshes/car.dae" scale="1 1 1"/>
+                    <mesh filename="file:///home/wu/code/ros2/Pure-tracking-slam-automatic-navigation-system/src/four_wheeled_vehicle/models/four_wheeled_vehicle/meshes/car.dae"/>
                 </geometry>
             </visual>

Commit message: 完善

File: src/four_wheeled_vehicle/urdf/vehicle/actuator/wheel.urdf.xacro (robot description, xacro)
@@ -29,5 +29,5 @@
                 <origin xyz="0 0 0" rpy="0 0 0"/>
                 <geometry>
-                    <mesh filename="file:///home/wu/code/ros2/Pure-tracking-slam-automatic-navigation-system/src/four_wheeled_vehicle/models/four_wheeled_vehicle/meshes/wheel_l.dae"/>
+                    <mesh filename="file://$(env HOME)/.gazebo/models/su7ultra/meshes/wheel_l.dae"/>
                 </geometry>
             </visual>
@@ -63,5 +63,5 @@
                 <origin xyz="0 0 0" rpy="0 0 0"/>
                 <geometry>
-                    <mesh filename="file:///home/wu/code/ros2/Pure-tracking-slam-automatic-navigation-system/src/four_wheeled_vehicle/models/four_wheeled_vehicle/meshes/wheel_r.dae"/>
+                    <mesh filename="file://$(env HOME)/.gazebo/models/su7ultra/meshes/wheel_r.dae"/>
                 </geometry>
             </visual>

File: src/four_wheeled_vehicle/urdf/vehicle/base.urdf.xacro (robot description, xacro)
@@ -16,5 +16,5 @@
                 <origin xyz="0 0 0" rpy="0 0 0"/>
                 <geometry>
-                    <mesh filename="file:///home/wu/code/ros2/Pure-tracking-slam-automatic-navigation-system/src/four_wheeled_vehicle/models/four_wheeled_vehicle/meshes/car.dae" scale="1 1 1"/>
+                    <mesh filename="file://$(env HOME)/.gazebo/models/su7ultra/meshes/car.dae" scale="1 1 1"/>
                 </geometry>
             </visual>
