Commit message: 将dae由绝对路径修改为不依赖用户名的方式

File: src/su7ultra_description/urdf/actuator/wheel.urdf.xacro (robot description, xacro)
@@ -29,5 +29,5 @@
                 <origin xyz="0 0 0" rpy="0 0 0"/>
                 <geometry>
-                    <mesh filename="file:///home/wu/.gazebo/models/su7ultra/meshes/wheel_l.dae"/>
+                    <mesh filename="file://$(env HOME)/.gazebo/models/su7ultra/meshes/wheel_l.dae"/>
                 </geometry>
             </visual>
@@ -63,5 +63,5 @@
                 <origin xyz="0 0 0" rpy="0 0 0"/>
                 <geometry>
-                    <mesh filename="file:///home/wu/.gazebo/models/su7ultra/meshes/wheel_r.dae"/>
+                    <mesh filename="file://$(env HOME)/.gazebo/models/su7ultra/meshes/wheel_r.dae"/>
                 </geometry>
             </visual>

File: src/su7ultra_description/urdf/base.urdf.xacro (robot description, xacro)
@@ -16,5 +16,5 @@
                 <origin xyz="0 0 0" rpy="0 0 0"/>
                 <geometry>
-                    <mesh filename="file:///home/wu/.gazebo/models/su7ultra/meshes/car.dae" scale="1 1 1"/>
+                    <mesh filename="file://$(env HOME)/.gazebo/models/su7ultra/meshes/car.dae" scale="1 1 1"/>
                 </geometry>
             </visual>

Commit message: 目前可以运行的版本

File: src/su7ultra_description/urdf/actuator/wheel.urdf.xacro (robot description, xacro)
@@ -29,5 +29,5 @@
                 <origin xyz="0 0 0" rpy="0 0 0"/>
                 <geometry>
-                    <mesh filename="file://$(env HOME)/.gazebo/models/su7ultra/meshes/wheel_l.dae"/>
+                    <mesh filename="file:///home/wu/.gazebo/models/su7ultra/meshes/wheel_l.dae"/>
                 </geometry>
             </visual>
@@ -63,5 +63,5 @@
                 <origin xyz="0 0 0" rpy="0 0 0"/>
                 <geometry>
-                    <mesh filename="file://$(env HOME)/.gazebo/models/su7ultra/meshes/wheel_r.dae"/>
+                    <mesh filename="file:///home/wu/.gazebo/models/su7ultra/meshes/wheel_r.dae"/>
                 </geometry>
             </visual>

File: src/su7ultra_description/urdf/base.urdf.xacro (robot description, xacro)
@@ -16,5 +16,5 @@
                 <origin xyz="0 0 0" rpy="0 0 0"/>
                 <geometry>
-                    <mesh filename="file://$(env HOME)/.gazebo/models/su7ultra/meshes/car.dae" scale="1 1 1"/>
+                    <mesh filename="file:///home/wu/.gazebo/models/su7ultra/meshes/car.dae" scale="1 1 1"/>
                 </geometry>
             </visual>
